Commit message: melodic

File: urdf/accessories/sensor_arch.urdf.xacro (robot description, xacro)
@@ -2,4 +2,5 @@
 <robot xmlns:xacro="http://ros.org/wiki/xacro" name="510_mm_sensor_arch">
     <xacro:macro name="sensor_arch" params="prefix parent size:=510 *origin">
+        <link name="${prefix}sensor_arch_base_link" />
         <!-- Spawn the sensor arch link -->
         <link name="${prefix}sensor_arch_mount_link">
@@ -7,5 +8,5 @@
              <visual>
                  <geometry>
-                     <mesh filename="package://ur5e_husky/meshes/accessories/${size}_mm_sensor_arch.dae" />
+                     <mesh filename="package://husky_description/meshes/accessories/${size}_mm_sensor_arch.dae" />
                  </geometry>
              </visual>
@@ -13,13 +14,18 @@
                  <origin xyz="0 0 0" rpy="0 0 0"/>
                  <geometry>
-                     <mesh filename="package://ur5e_husky/meshes/accessories/${size}_mm_sensor_arch.dae" />
+                     <mesh filename="package://husky_description/meshes/accessories/${size}_mm_sensor_arch.dae" />
                  </geometry>
              </collision>
         </link>
+        <joint name="${prefix}sensor_arch_base_link_joint" type="fixed">
+            <parent link="${parent}" />
+            <child link="${prefix}sensor_arch_base_link" />
+            <xacro:insert_block name="origin" />
+        </joint>
         <!-- Attach the sensor arch to the top plate -->
         <joint name="${prefix}sensor_arch_mount" type="fixed">
-             <xacro:insert_block name="origin"/>
-             <parent link="${parent}"/>
+             <parent link="${prefix}sensor_arch_base_link"/>
              <child link="${prefix}sensor_arch_mount_link"/>
+             <origin xyz="0 0 ${size/1000}" rpy="0 0 0" />
         </joint>
     </xacro:macro>

File: urdf/accessories/sick_lms1xx_mount.urdf.xacro (robot description, xacro)
@@ -33,5 +33,5 @@
         <geometry>
           <!-- Origin of this mesh is the base of the bracket. -->
-          <mesh filename="package://ur5e_husky/meshes/accessories/lms1xx_mount.dae" />
+          <mesh filename="package://husky_description/meshes/accessories/lms1xx_mount.dae" />
         </geometry>
       </visual>

File: urdf/decorations.urdf.xacro (robot description, xacro)
@@ -30,6 +30,8 @@
   <material name="red"><color rgba="1.0 0.0 0.0 1.0" /></material>
   <xacro:macro name="husky_decorate">
+    <xacro:property name="husky_front_bumper_enable" value="$(optenv HUSKY_FRONT_BUMPER 1)" />
+    <xacro:property name="husky_rear_bumper_enable"  value="$(optenv HUSKY_REAR_BUMPER 1)" />
     <xacro:property name="husky_front_bumper_extend" value="$(optenv HUSKY_FRONT_BUMPER_EXTEND 0)" />
-    <xacro:property name="husky_rear_bumper_extend" value="$(optenv HUSKY_REAR_BUMPER_EXTEND 0)" />
+    <xacro:property name="husky_rear_bumper_extend"  value="$(optenv HUSKY_REAR_BUMPER_EXTEND 0)" />
     <!-- Spawn Husky chassis -->
     <link name="top_chassis_link">
@@ -37,5 +39,5 @@
         <origin xyz="0 0 0" rpy="0 0 0" />
         <geometry>
-          <mesh filename="package://ur5e_husky/meshes/top_chassis.dae" />
+          <mesh filename="package://husky_description/meshes/top_chassis.dae" />
         </geometry>
       </visual>
@@ -51,5 +53,5 @@
         <visual>
           <geometry>
-            <mesh filename="package://ur5e_husky/meshes/user_rail.dae" />
+            <mesh filename="package://husky_description/meshes/user_rail.dae" />
           </geometry>
         </visual>
@@ -63,58 +65,62 @@
     </xacro:if>
     <!-- Spawn front bumper link -->
-    <link name="front_bumper_link">
-      <visual>
-        <geometry>
-          <mesh filename="package://ur5e_husky/meshes/bumper.dae" />
-        </geometry>
-      </visual>
-    </link>
-    <!-- Attach front bumper -->
-    <joint name="front_bumper" type="fixed">
-      <origin xyz="${0.48 + husky_front_bumper_extend} 0 0.091" rpy="0 0 0" />
-      <parent link="base_link" />
-      <child link="front_bumper_link" />
-    </joint>
-    <xacro:if value="${husky_front_bumper_extend}">
-      <link name="front_bumper_extension_link">
-          <visual>
-              <geometry>
-                  <mesh filename="package://ur5e_husky/meshes/bumper_extension.dae" />
-              </geometry>
-          </visual>
+    <xacro:if value="${husky_front_bumper_enable}">
+      <link name="front_bumper_link">
+        <visual>
+          <geometry>
+            <mesh filename="package://husky_description/meshes/bumper.dae" />
+          </geometry>
+        </visual>
       </link>
-      <joint name="front_bumper_extension" type="fixed">
+      <!-- Attach front bumper -->
+      <joint name="front_bumper" type="fixed">
         <origin xyz="${0.48 + husky_front_bumper_extend} 0 0.091" rpy="0 0 0" />
         <parent link="base_link" />
-        <child link="front_bumper_extension_link" />
+        <child link="front_bumper_link" />
       </joint>
+      <xacro:if value="${husky_front_bumper_extend}">
+        <link name="front_bumper_extension_link">
+            <visual>
+                <geometry>
+                    <mesh filename="package://husky_description/meshes/bumper_extension.dae" />
+                </geometry>
+            </visual>
+        </link>
+        <joint name="front_bumper_extension" type="fixed">
+          <origin xyz="${0.48 + husky_front_bumper_extend} 0 0.091" rpy="0 0 0" />
+          <parent link="base_link" />
+          <child link="front_bumper_extension_link" />
+        </joint>
+      </xacro:if>
     </xacro:if>
     <!-- Spawn rear bumper link -->
-    <link name="rear_bumper_link">
-      <visual>
-        <geometry>
-          <mesh filename="package://ur5e_husky/meshes/bumper.dae" />
-        </geometry>
-      </visual>
-    </link>
-    <!-- Attach rear bumper -->
-    <joint name="rear_bumper" type="fixed">
-      <origin xyz="${-0.48 - husky_rear_bumper_extend} 0 0.091" rpy="0 0 ${M_PI}" />
-      <parent link="base_link" />
-      <child link="rear_bumper_link" />
-    </joint>
-    <xacro:if value="${husky_rear_bumper_extend}">
-      <link name="rear_bumper_extension_link">
-          <visual>
-              <geometry>
-                  <mesh filename="package://ur5e_husky/meshes/bumper_extension.dae" />
-              </geometry>
-          </visual>
+    <xacro:if value="${husky_rear_bumper_enable}">
+      <link name="rear_bumper_link">
+        <visual>
+          <geometry>
+            <mesh filename="package://husky_description/meshes/bumper.dae" />
+          </geometry>
+        </visual>
       </link>
-      <joint name="rear_bumper_extension" type="fixed">
+      <!-- Attach rear bumper -->
+      <joint name="rear_bumper" type="fixed">
         <origin xyz="${-0.48 - husky_rear_bumper_extend} 0 0.091" rpy="0 0 ${M_PI}" />
         <parent link="base_link" />
-        <child link="rear_bumper_extension_link" />
+        <child link="rear_bumper_link" />
       </joint>
+      <xacro:if value="${husky_rear_bumper_extend}">
+        <link name="rear_bumper_extension_link">
+            <visual>
+                <geometry>
+                    <mesh filename="package://husky_description/meshes/bumper_extension.dae" />
+                </geometry>
+            </visual>
+        </link>
+        <joint name="rear_bumper_extension" type="fixed">
+          <origin xyz="${-0.48 - husky_rear_bumper_extend} 0 0.091" rpy="0 0 ${M_PI}" />
+          <parent link="base_link" />
+          <child link="rear_bumper_extension_link" />
+        </joint>
+      </xacro:if>
     </xacro:if>
     <xacro:if value="$(optenv HUSKY_TOP_PLATE_ENABLED true)">
@@ -125,5 +131,5 @@
             <origin xyz="0 0 0" rpy="0 0 0" />
             <geometry>
-              <mesh filename="package://ur5e_husky/meshes/large_top_plate.dae" />
+              <mesh filename="package://husky_description/meshes/large_top_plate.dae" />
             </geometry>
           </visual>
@@ -131,5 +137,5 @@
             <origin xyz="0 0 0" rpy="0 0 0"/>
             <geometry>
-              <mesh filename="package://ur5e_husky/meshes/large_top_plate_collision.stl" />
+              <mesh filename="package://husky_description/meshes/large_top_plate_collision.stl" />
             </geometry>
           </collision>
@@ -159,5 +165,5 @@
             <origin xyz="0 0 0" rpy="0 0 0" />
             <geometry>
-              <mesh filename="package://ur5e_husky/meshes/top_plate.dae" />
+              <mesh filename="package://husky_description/meshes/top_plate.dae" />
             </geometry>
           </visual>
@@ -165,5 +171,5 @@
             <origin xyz="0 0 0" rpy="0 0 0"/>
             <geometry>
-              <mesh filename="package://ur5e_husky/meshes/top_plate.stl" />
+              <mesh filename="package://husky_description/meshes/top_plate.stl" />
             </geometry>
           </collision>

File: urdf/husky.urdf.xacro (robot description, xacro)
@@ -22,8 +22,14 @@
 -->
 <robot name="husky" xmlns:xacro="http://ros.org/wiki/xacro">
-  <xacro:arg name="laser_enabled" default="false" />
+  <xacro:arg name="laser_enabled" default="$(optenv HUSKY_LMS1XX_ENABLED 0)" />
   <xacro:arg name="laser_xyz" default="$(optenv HUSKY_LMS1XX_XYZ 0.2206 0.0 0.00635)" />
   <xacro:arg name="laser_rpy" default="$(optenv HUSKY_LMS1XX_RPY 0.0 0.0 0.0)" />
-  <xacro:arg name="realsense_enabled" default="false" />
+  <xacro:arg name="laser_secondary_enabled" default="$(optenv HUSKY_LMS1XX_SECONDARY_ENABLED 0)" />
+  <xacro:arg name="laser_secondary_xyz" default="$(optenv HUSKY_LMS1XX_SECONDARY_XYZ -0.2206 0.0 0.00635)" />
+  <xacro:arg name="laser_secondary_rpy" default="$(optenv HUSKY_LMS1XX_SECONDARY_RPY 0.0 0.0 3.14159)" />
+  <xacro:arg name="laser_3d_enabled" default="$(optenv HUSKY_LASER_3D_ENABLED 0)" />
+  <xacro:arg name="laser_3d_xyz" default="$(optenv HUSKY_LASER_3D_XYZ 0 0 0)" />
+  <xacro:arg name="laser_3d_rpy" default="$(optenv HUSKY_LASER_3D_RPY 0 0 0)" />
+  <xacro:arg name="realsense_enabled" default="$(optenv HUSKY_REALSENSE_ENABLED 0)" />
   <xacro:arg name="realsense_xyz" default="$(optenv HUSKY_REALSENSE_XYZ 0 0 0)" />
   <xacro:arg name="realsense_rpy" default="$(optenv HUSKY_REALSENSE_RPY 0 0 0)" />
@@ -31,12 +37,17 @@
   <xacro:property name="husky_front_bumper_extend" value="$(optenv HUSKY_FRONT_BUMPER_EXTEND 0)" />
   <xacro:property name="husky_rear_bumper_extend" value="$(optenv HUSKY_REAR_BUMPER_EXTEND 0)" />
-  <xacro:arg name="robot_namespace" default="/" />
-  <xacro:arg name="urdf_extras" default="empty.urdf" />
+  <!-- Height of the sensor arch in mm.  Must be either 510 or 300 -->
+  <xacro:arg name="sensor_arch_height"  default="$(optenv HUSKY_SENSOR_ARCH_HEIGHT 510)" />
+  <xacro:arg name="sensor_arch"         default="$(optenv HUSKY_SENSOR_ARCH 0)" />
+  <xacro:arg name="robot_namespace" default="$(optenv ROBOT_NAMESPACE /)" />
+  <xacro:arg name="urdf_extras" default="$(optenv HUSKY_URDF_EXTRAS empty.urdf)" />
+  <xacro:arg name="cpr_urdf_extras" default="$(optenv CPR_URDF_EXTRAS empty.urdf)" />
   <!-- Included URDF/XACRO Files -->
-  <xacro:include filename="$(find ur5e_husky)/urdf/decorations.urdf.xacro" />
-  <xacro:include filename="$(find ur5e_husky)/urdf/wheel.urdf.xacro" />
-  <xacro:include filename="$(find ur5e_husky)/urdf/accessories/intel_realsense.urdf.xacro"/>
-  <xacro:include filename="$(find ur5e_husky)/urdf/accessories/sick_lms1xx_mount.urdf.xacro"/>
-  <xacro:include filename="$(find ur5e_husky)/urdf/accessories/sensor_arch.urdf.xacro"/>
+  <xacro:include filename="$(find husky_description)/urdf/decorations.urdf.xacro" />
+  <xacro:include filename="$(find husky_description)/urdf/wheel.urdf.xacro" />
+  <xacro:include filename="$(find husky_description)/urdf/accessories/intel_realsense.urdf.xacro"/>
+  <xacro:include filename="$(find husky_description)/urdf/accessories/sick_lms1xx_mount.urdf.xacro"/>
+  <xacro:include filename="$(find husky_description)/urdf/accessories/sensor_arch.urdf.xacro"/>
+  <xacro:include filename="$(find husky_description)/urdf/accessories/vlp16_mount.urdf.xacro"/>
   <xacro:property name="M_PI" value="3.14159"/>
   <!-- Base Size -->
@@ -56,5 +67,5 @@
       <origin xyz="0 0 0" rpy="0 0 0" />
       <geometry>
-        <mesh filename="package://ur5e_husky/meshes/base_link.dae" />
+        <mesh filename="package://husky_description/meshes/base_link.dae" />
       </geometry>
     </visual>
@@ -116,4 +127,7 @@
   </xacro:husky_wheel>
   <xacro:husky_decorate />
+  <!--
+    Add the primary and secondary lasers
+  -->
   <xacro:if value="$(arg laser_enabled)">
     <xacro:sick_lms1xx_mount prefix="base"/>
@@ -125,24 +139,42 @@
     </joint>
   </xacro:if>
+  <xacro:if value="$(arg laser_secondary_enabled)">
+    <xacro:sick_lms1xx_mount prefix="rear"/>
+    <xacro:sick_lms1xx frame="rear_laser" topic="rear/scan" robot_namespace="$(arg robot_namespace)"/>
+    <joint name="laser_secondary_mount_joint" type="fixed">
+      <origin xyz="$(arg laser_secondary_xyz)" rpy="$(arg laser_secondary_rpy)" />
+      <parent link="top_plate_link" />
+      <child link="rear_laser_mount" />
+    </joint>
+  </xacro:if>
   <!--
-    top sensor arch; include this if we have realsense enabled
-    keep this as a property to make it easier to add multiple conditions, should we need
-    the top bar for any additional sensors in the future
+    Add the main sensor arch if the user has specifically enabled it, or if a sensor
+    requires it for mounting
   -->
-  <xacro:property name="topbar_needed_realsense" value="$(arg realsense_enabled)" />
-  <xacro:if value="${topbar_needed_realsense}">
-    <xacro:sensor_arch prefix="" parent="top_plate_link">
-      <origin xyz="-0.35 0 0.51" rpy="0 0 -3.14"/>
-    </xacro:sensor_arch>
-  </xacro:if>
-  <!-- add the intel realsense to the topbar if needed -->
+  <xacro:property name="sensorbar_user_enabled"     value="$(arg sensor_arch)" />
+  <xacro:property name="sensorbar_needed_realsense" value="$(arg realsense_enabled)" />
+  <xacro:property name="sensorbar_needed_lidar"     value="$(arg laser_3d_enabled)" />
+  <xacro:if value="${sensorbar_needed_realsense or sensorbar_user_enabled or sensorbar_needed_lidar}">
+    <xacro:sensor_arch prefix="" parent="top_plate_link" size="$(arg sensor_arch_height)">
+        <origin xyz="$(optenv HUSKY_SENSOR_ARCH_OFFSET 0 0 0)" rpy="$(optenv HUSKY_SENSOR_ARCH_RPY 0 0 0)"/>
+      </xacro:sensor_arch>
+  </xacro:if>
+  <!-- add the intel realsense to the sensor arch if needed -->
   <xacro:if value="$(arg realsense_enabled)">
     <link name="realsense_mountpoint"/>
     <joint name="realsense_mountpoint_joint" type="fixed">
-      <origin xyz="0 0 0" rpy="0 0 -3.14159" />
+      <origin xyz="$(arg realsense_xyz)" rpy="$(arg realsense_rpy)" />
       <parent link="$(arg realsense_mount)"/>
       <child link="realsense_mountpoint" />
     </joint>
     <xacro:intel_realsense_mount prefix="camera" topic="realsense" parent_link="realsense_mountpoint"/>
+  </xacro:if>
+  <!--
+    Add the 3d laser to the sensor arch if needed
+  -->
+  <xacro:if value="$(arg laser_3d_enabled)">
+    <xacro:vlp16_mount prefix="" parent_link="sensor_arch_mount_link" topic="$(optenv HUSKY_LASER_3D_TOPIC points)">
+      <origin xyz="$(arg laser_3d_xyz)" rpy="$(arg laser_3d_rpy)" />
+    </xacro:vlp16_mount>
   </xacro:if>
   <gazebo>
@@ -183,3 +215,5 @@
   <!-- Optional custom includes. -->
   <xacro:include filename="$(arg urdf_extras)" />
+  <!-- Optional for Clearpath internal softwares -->
+  <xacro:include filename="$(arg cpr_urdf_extras)" />
 </robot>

File: urdf/wheel.urdf.xacro (robot description, xacro)
@@ -32,5 +32,5 @@
 				<origin xyz="0 0 0" rpy="0 0 0" />
 				<geometry>
-					<mesh filename="package://ur5e_husky/meshes/wheel.dae" />
+					<mesh filename="package://husky_description/meshes/wheel.dae" />
 				</geometry>
 			</visual>
